File: keychain.kicad_pcb (KiCad board)
At the start: 2 copper layers, 100 x 20 mm, 2 parts, among them U1 ST25DV04K-JFR6D3

Commit message: Test production
Parts:
- added G1: LOGO, LOGO, F.Cu at (175.0, 94.5)
- added G2: LOGO, LOGO, B.Cu at (175.0, 94.5)
